File: Rocket_v1.kicad_pcb (KiCad board)
At the start: 2 copper layers, 30 x 115.5 mm, 6 parts, among them J4 Conn_01x02_Socket, SW1 SW_SPDT

Commit message: Final Computer layout for all Sensors
Parts:
- moved JMPU6050 13.4 mm to (133.9, 69.5), turned to 90 degrees
- renumbered JSGP30 to JMPU6050
Routing:
- net /+3V3: track 145.3 -> 125.1 mm
- net /I2C_SCL: track 198.4 -> 187.2 mm
Changed lines of the file:
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@@
 	(footprint "Connector_PinHeader_2.54mm:PinHeader_1x04_P2.54mm_Vertical"
 		(layer "F.Cu")
-		(at 142.5 59.19)
+		(at 133.92 69.5 90)
 		(descr "Through hole straight pin header, 1x04, 2.54mm pitch, single row")
 		(tags "Through hole pin header THT 1x04 2.54mm single row")
-		(property "Reference" "JSGP30"
-			(at 0 -2.38 0)
+		(property "Reference" "JMPU6050"
+			(at -2.81 4.81 180)
 			(layer "F.SilkS")
 			(effects
@@
 		)
 		(property "Value" "Conn_01x04_Pin"
-			(at 0 10 0)
+			(at 0 10 90)
 			(layer "F.Fab")
 			(effects
@@
 		)
 		(property "Datasheet" ""
-			(at 0 0 0)
+			(at 0 0 90)
 			(layer "F.Fab")
 			(hide yes)
@@
 		)
 		(property "Description" "Generic connector, single row, 01x04, script generated"
-			(at 0 0 0)
+			(at 0 0 90)
 			(layer "F.Fab")
 			(hide yes)
@@
 		)
 		(property "KiLib_Generator" "connector/pin_header_socket"
-			(at 0 0 0)
+			(at 0 0 90)
 			(layer "F.SilkS")
 			(hide yes)
@@
 		)
 		(fp_line
+			(start 1.38 1.27)
+			(end 1.38 9)
+			(stroke
+				(width 0.12)
+				(type solid)
+			)
+			(layer "F.SilkS")
+		)
+		(fp_line
+			(start -1.38 1.27)
+			(end 1.38 1.27)
+			(stroke
+				(width 0.12)
+				(type solid)
+			)
+			(layer "F.SilkS")
+		)
+		(fp_line
 			(start -1.38 1.27)
 			(end -1.38 9)
@@
 		)
 		(fp_line
-			(start -1.38 1.27)
-			(end 1.38 1.27)
-			(stroke
-				(width 0.12)
-				(type solid)
-			)
-			(layer "F.SilkS")
-		)
-		(fp_line
 			(start -1.38 9)
-			(end 1.38 9)
-			(stroke
-				(width 0.12)
-				(type solid)
-			)
-			(layer "F.SilkS")
-		)
-		(fp_line
-			(start 1.38 1.27)
 			(end 1.38 9)
 			(stroke
@@
 		)
 		(fp_line
+			(start 1.27 -1.27)
+			(end 1.27 8.89)
+			(stroke
+				(width 0.1)
+				(type solid)
+			)
+			(layer "F.Fab")
+		)
+		(fp_line
+			(start -0.635 -1.27)
+			(end 1.27 -1.27)
+			(stroke
+				(width 0.1)
+				(type solid)
+			)
+			(layer "F.Fab")
+		)
+		(fp_line
 			(start -1.27 -0.635)
 			(end -0.635 -1.27)
@@
 		)
 		(fp_line
+			(start 1.27 8.89)
+			(end -1.27 8.89)
+			(stroke
+				(width 0.1)
+				(type solid)
+			)
+			(layer "F.Fab")
+		)
+		(fp_line
 			(start -1.27 8.89)
 			(end -1.27 -0.635)
@@
 			(layer "F.Fab")
 		)
-		(fp_line
-			(start -0.635 -1.27)
-			(end 1.27 -1.27)
-			(stroke
-				(width 0.1)
-				(type solid)
-			)
-			(layer "F.Fab")
-		)
-		(fp_line
-			(start 1.27 -1.27)
-			(end 1.27 8.89)
-			(stroke
-				(width 0.1)
-				(type solid)
-			)
-			(layer "F.Fab")
-		)
-		(fp_line
-			(start 1.27 8.89)
-			(end -1.27 8.89)
-			(stroke
-				(width 0.1)
-				(type solid)
-			)
-			(layer "F.Fab")
-		)
 		(fp_text user "${REFERENCE}"
 			(at 0 3.81 90)
@@
 		)
 		(pad "1" thru_hole rect
-			(at 0 0)
+			(at 0 0 90)
 			(size 1.7 1.7)
 			(drill 1)
@@
 		)
 		(pad "2" thru_hole circle
-			(at 0 2.54)
+			(at 0 2.54 90)
 			(size 1.7 1.7)
 			(drill 1)
@@
 		)
 		(pad "3" thru_hole circle
-			(at 0 5.08)
+			(at 0 5.08 90)
 			(size 1.7 1.7)
 			(drill 1)
@@
 		)
 		(pad "4" thru_hole circle
-			(at 0 7.62)
+			(at 0 7.62 90)
 			(size 1.7 1.7)
 			(drill 1)
@@
 	)
 	(segment
-		(start 128.2 70.8)
-		(end 134.73 64.27)
-		(width 0.6)
-		(layer "F.Cu")
-		(net "/I2C_SCL")
-	)
-	(segment
 		(start 128.2 168.2)
 		(end 128.2 107)
@@
 	)
 	(segment
+		(start 128.2 92.5)
+		(end 128.2 80.3)
+		(width 0.6)
+		(layer "F.Cu")
+		(net "/I2C_SCL")
+	)
+	(segment
 		(start 156 157.5)
 		(end 156 170)
@@
 	)
 	(segment
-		(start 128.2 92.5)
-		(end 128.2 70.8)
-		(width 0.6)
-		(layer "F.Cu")
-		(net "/I2C_SCL")
-	)
-	(segment
 		(start 154.2 155.7)
 		(end 156 157.5)
@@
 	)
 	(segment
-		(start 134.73 64.27)
-		(end 142.5 64.27)
-		(width 0.6)
-		(layer "F.Cu")
-		(net "/I2C_SCL")
-	)
-	(segment
 		(start 156 170)
 		(end 155.3 170.7)
@@
 	)
 	(segment
+		(start 128.2 80.3)
+		(end 139 69.5)
+		(width 0.6)
+		(layer "F.Cu")
+		(net "/I2C_SCL")
+	)
+	(segment
 		(start 142.27 82.5)
 		(end 142.5 82.27)
@@
 	)
 	(segment
-		(start 156 92)
-		(end 156 80.31)
-		(width 0.6)
-		(layer "F.Cu")
-		(net "/I2C_SDA")
-	)
-	(segment
 		(start 149.69 92)
 		(end 142.5 84.81)
@@
 	)
 	(segment
-		(start 156 80.31)
-		(end 142.5 66.81)
-		(width 0.6)
-		(layer "F.Cu")
-		(net "/I2C_SDA")
-	)
-	(segment
 		(start 153.84 153.16)
 		(end 156 151)
@@
 	)
 	(segment
+		(start 156 80)
+		(end 145.5 69.5)
+		(width 0.6)
+		(layer "F.Cu")
+		(net "/I2C_SDA")
+	)
+	(segment
+		(start 145.5 69.5)
+		(end 141.54 69.5)
+		(width 0.6)
+		(layer "F.Cu")
+		(net "/I2C_SDA")
+	)
+	(segment
 		(start 156 151)
 		(end 156 109)
@@
 	)
 	(segment
+		(start 156 92)
+		(end 156 80)
+		(width 0.6)
+		(layer "F.Cu")
+		(net "/I2C_SDA")
+	)
+	(segment
 		(start 133.9 158.24)
 		(end 130.74 158.24)
@@
 	)
 	(segment
-		(start 129 83)
-		(end 129 62)
+		(start 131.81 94.69)
+		(end 142.4 94.69)
 		(width 0.6)
 		(layer "B.Cu")
@@
 	)
 	(segment
-		(start 131.81 94.69)
-		(end 142.4 94.69)
+		(start 129 83)
+		(end 133.92 78.08)
 		(width 0.6)
 		(layer "B.Cu")
@@
 	)
 	(segment
-		(start 131.81 59.19)
-		(end 142.5 59.19)
+		(start 129 83)
+		(end 134.81 77.19)
 		(width 0.6)
 		(layer "B.Cu")
@@
 	)
 	(segment
-		(start 129 83)
-		(end 134.81 77.19)
+		(start 129 156.5)
+		(end 129 97.5)
 		(width 0.6)
 		(layer "B.Cu")
@@
 	)
 	(segment
-		(start 129 62)
-		(end 131.81 59.19)
+		(start 129 97.5)
+		(end 131.81 94.69)
 		(width 0.6)
 		(layer "B.Cu")
@@
 	)
 	(segment
-		(start 129 156.5)
-		(end 129 97.5)
+		(start 133.92 78.08)
+		(end 133.92 69.5)
 		(width 0.6)
 		(layer "B.Cu")
-		(net "/+3V3")
-	)
-	(segment
-		(start 129 97.5)
-		(end 131.81 94.69)
-		(width 0.6)
-		(layer "B.Cu")
