File: Buzzard-Avionics.kicad_pcb (KiCad board)
At the start: 2 copper layers, 30 x 115.5 mm, 6 parts, among them J4 Conn_01x02_Socket, SW1 SW_SPDT

Commit message: Releases/Mayor added
Parts:
- moved JMPU6050 77.9 mm to (196.5, 115.9), turned to 0 degrees
- moved JMPU6050 66.2 mm to (188.8, 124.5), turned to -90 degrees
- moved A1 64.3 mm to (97.6, 133.7), turned to 90 degrees
- moved BMP280 41.5 mm to (171.3, 124.4), turned to -90 degrees
- moved SW1 19.6 mm to (152.5, 114.9), turned to -90 degrees
- moved J4 19.0 mm to (152.1, 132.9), turned to 90 degrees
Other:
- board size 30 x 115.5 mm -> 115.5 x 30 mm

Commit message: Naming Error on the Board fixed
Parts:
- renumbered JMPU6050 to JSGP30, JMPU6050 to MPU6050
Changed lines of the file:
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@@
 		(property ki_fp_filters "Connector*:*_1x??_*")
 		(sheetname "/")
-		(sheetfile "Rakete_v1.kicad_sch")
+		(sheetfile "Buzzard-Avionics.kicad_sch")
 		(units
 			(unit
@@
 		)
 		(sheetname "/")
-		(sheetfile "Rakete_v1.kicad_sch")
+		(sheetfile "Buzzard-Avionics.kicad_sch")
 		(units
 			(unit
@@
 		(property ki_fp_filters "RaspberryPi?Pico?Common* RaspberryPi?Pico?SMD*")
 		(sheetname "/")
-		(sheetfile "Rakete_v1.kicad_sch")
+		(sheetfile "Buzzard-Avionics.kicad_sch")
 		(units
 			(unit
@@
 		(descr "Through hole straight pin header, 1x04, 2.54mm pitch, single row")
 		(tags "Through hole pin header THT 1x04 2.54mm single row")
-		(property "Reference" "JMPU6050"
-			(at -2.81 4.81 90)
+		(property "Reference" "JSGP30"
+			(at -5.5 8.58 90)
 			(layer "F.SilkS")
 			(effects
@@
 		(property ki_fp_filters "Connector*:*_1x??_*")
 		(sheetname "/")
-		(sheetfile "Rakete_v1.kicad_sch")
+		(sheetfile "Buzzard-Avionics.kicad_sch")
 		(units
 			(unit
@@
 		(tags "Through hole pin header THT 1x04 2.54mm single row")
 		(property "Reference" "BMP280"
-			(at 0 -2.38 90)
+			(at 0 -2.38 270)
 			(layer "F.SilkS")
 			(effects
@@
 		(property ki_fp_filters "Connector*:*_1x??_*")
 		(sheetname "/")
-		(sheetfile "Rakete_v1.kicad_sch")
+		(sheetfile "Buzzard-Avionics.kicad_sch")
 		(units
 			(unit
@@
 		(descr "Through hole straight pin header, 1x04, 2.54mm pitch, single row")
 		(tags "Through hole pin header THT 1x04 2.54mm single row")
-		(property "Reference" "JMPU6050"
-			(at 0 -2.38 90)
+		(property "Reference" "MPU6050"
+			(at -4 -5.19 270)
 			(layer "F.SilkS")
 			(effects
@@
 		(property ki_fp_filters "Connector*:*_1x??_*")
 		(sheetname "/")
-		(sheetfile "Rakete_v1.kicad_sch")
+		(sheetfile "Buzzard-Avionics.kicad_sch")
 		(units
 			(unit
