File: Buzzard-Avionics.kicad_sch (KiCad schematic)
At the start: 6 parts, among them J4 Conn_01x02_Socket, SW1 SW_SPDT

Commit message: Schematic update
Parts:
- renumbered JMPU6050 to MPU6050
Changed lines of the file:
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@@
 		)
 		(instances
-			(project "Rakete_v1"
+			(project "Buzzard-Avionics"
 				(path "/c8b6c309-6573-422c-a8ed-173ce712d251"
 					(reference "A1")
@@
 		)
 		(instances
-			(project "Rakete_v1"
+			(project "Buzzard-Avionics"
 				(path "/c8b6c309-6573-422c-a8ed-173ce712d251"
 					(reference "J4")
@@
 		)
 		(instances
-			(project "Rakete_v1"
+			(project "Buzzard-Avionics"
 				(path "/c8b6c309-6573-422c-a8ed-173ce712d251"
 					(reference "SW1")
@@
 		)
 		(instances
-			(project "Rakete_v1"
+			(project "Buzzard-Avionics"
 				(path "/c8b6c309-6573-422c-a8ed-173ce712d251"
 					(reference "#FLG01")
@@
 		(dnp no)
 		(fields_autoplaced yes)
-		(property "Reference" "JMPU6050"
+		(property "Reference" "MPU6050"
 			(at 66.675 139.7 0)
 			(show_name no)
@@
 		)
 		(instances
-			(project "Rakete_v1"
-				(path "/c8b6c309-6573-422c-a8ed-173ce712d251"
-					(reference "JMPU6050")
+			(project "Buzzard-Avionics"
+				(path "/c8b6c309-6573-422c-a8ed-173ce712d251"
+					(reference "MPU6050")
 					(unit 1)
 				)
@@
 		)
 		(instances
-			(project "Rakete_v1"
+			(project "Buzzard-Avionics"
 				(path "/c8b6c309-6573-422c-a8ed-173ce712d251"
 					(reference "JSGP30")
@@
 		)
 		(instances
-			(project "Rakete_v1"
+			(project "Buzzard-Avionics"
 				(path "/c8b6c309-6573-422c-a8ed-173ce712d251"
 					(reference "BMP280")
